File: pcb/integrated/integrated.kicad_pcb (KiCad board)
At the start: 4 copper layers, 200 x 100 mm, 270 parts, among them J10001 Conn_01x02_Female, J1001 mounting-hole-grounded, J1002 mounting-hole-grounded, J1003 mounting-hole-grounded, J1004 mounting-hole-grounded, J3001 Conn_01x04_Male, J3002 Conn_01x06_Male, J5001 Conn_Coaxial, J8001 Conn_01x02_Female, Q10001 F423MR12W1M1B11BOMA1, Q8001 Q_NMOS_GDS, Q8002 Q_NMOS_GDS, U11001 UCC5350SB, U11002 R15P21503D, U12001 UCC5350SB, U12002 R15P21503D, U13001 UCC5350SB, U13002 R15P21503D, U14001 UCC5350SB, U14002 R15P21503D, U3001 XC7S25-L1FTGB196, U3002 S25FL127SABN, U3003 74AVC4TD245BQ, U5001 74LVC1G3157GW, U5002 TLV3501AIDBVR, U5003 74LVC1G3157GW, U5004 MCP6561-OT, U6001 SG3225, U6002 AD9609, U7001 AFBR-1624Z, U7002 AFBR-2624Z, U8001 SN74LVC1T45DBV, U8002 ADuM5230, U8003 ACS730, U9001 EC6AW, U9002 RAC10, U9003 TPS82140, U9004 TPS82140, U9005 TPS735, U9006 TPS735

Commit message: schematic fixes and component placement
Parts:
- removed FB4001, FB4002, FB6001: Ferrite_Bead, Inductor_SMD:L_0805_2012Metric
- added C8005: 0.47u, Capacitor_SMD:C_0402_1005Metric, F.Cu at (27.8, -34.2)
- added C9017: 0.47u, Capacitor_SMD:C_1812_4532Metric, F.Cu at (100.8, 75.8)
- added C9018: 470u, Capacitor_THT:CP_Radial_D10.0mm_P5.00mm, F.Cu at (91.0, 58.8)
- added C9019: 470u, Capacitor_THT:CP_Radial_D10.0mm_P5.00mm, F.Cu at (80.0, 58.8)
- added J1005: mounting-hole-grounded, wbraun_smd:M3-tight-fit-pan-head, F.Cu at (105.0, 54.5)
- added J1006: mounting-hole-grounded, wbraun_smd:M3-tight-fit-pan-head, F.Cu at (105.0, 145.5)
- added R8013: 10k, Resistor_SMD:R_0603_1608Metric, F.Cu at (28.3, -36.5)
- added R9007: 0, Resistor_SMD:R_0805_2012Metric, F.Cu at (36.7, 82.7)
- added R9008: 0, Resistor_SMD:R_0805_2012Metric, F.Cu at (36.7, 85.7)
- added R9009: 0, Resistor_SMD:R_0805_2012Metric, F.Cu at (41.1, 82.7)
- added R9010: 0, Resistor_SMD:R_0805_2012Metric, F.Cu at (104.8, 136.5)
- C4006, C5008, C5009, C6005, C6009, C6011, C6013: moved to B.Cu
- C9001: value 1u -> 0.47u; footprint Capacitor_SMD:C_0805_2012Metric -> Capacitor_SMD:C_1812_4532Metric
- C9002, C9003, C9004, C9005: footprint Capacitor_SMD:C_0805_2012Metric -> Capacitor_SMD:C_1206_3216Metric
- C9007, C9008: footprint Capacitor_SMD:C_0805_2012Metric -> Capacitor_SMD:C_0402_1005Metric
- C9011, C9012, C9015, C9016: footprint Capacitor_SMD:C_0402_1005Metric -> Capacitor_SMD:C_0603_1608Metric
- U8001: value SN74LVC1T45DBV -> 74LVC2T45DC; footprint Package_TO_SOT_SMD:SOT-23-6 -> Package_SO:VSSOP-8_2.3x2mm_P0.5mm
- moved C9010 209.7 mm to (83.8, 99.5), turned to 180 degrees
- moved R9001 208.4 mm to (76.5, 96.5), turned to 270 degrees
- moved C6001 181.7 mm to (94.5, 137.2), turned to 180 degrees
- moved C5005 178.4 mm to (72.5, 137.5)
- moved C6008 178.3 mm to (84.5, 135.0)
- moved U6001 177.2 mm to (94.5, 134.8), turned to 90 degrees
- moved C6002 176.2 mm to (94.5, 138.2), turned to 180 degrees
- moved C6009 174.4 mm to (90.5, 130.5)
- moved C6006 173.7 mm to (84.5, 133.9)
- moved C5016 173.2 mm to (87.5, 143.5)
- moved C5015 172.3 mm to (84.8, 146.5), turned to 90 degrees
- moved R5017 172.2 mm to (91.2, 144.8), turned to 270 degrees
- moved C6011 171.6 mm to (87.0, 127.5)
- moved C5017 170.4 mm to (87.5, 142.5)
- moved R5007 170.3 mm to (67.5, 134.0), turned to 180 degrees
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Connections:
- net SUPPLY_EN renamed SUPPLY_EN1
- C3003 pad 1: +3V3D -> +3V3
- C3004 pad 1: +3V3D -> +3V3
- C4003 pad 1: +1V8D -> +1V8
- C4004 pad 1: +3V3D -> +3V3
- C4007 pad 1: +1V8D -> +1V8
- C4008 pad 1: +3V3D -> +3V3
- C4009 pad 1: +3V3D -> +3V3
- C4010 pad 1: +1V8D -> +1V8
- C4013 pad 1: +3V3D -> +3V3
- C4014 pad 1: +3V3D -> +3V3
- C4015 pad 1: +1V8D -> +1V8
- C4017 pad 1: +3V3D -> +3V3
- C4018 pad 1: +3V3D -> +3V3
- C4020 pad 1: +3V3D -> +3V3
- C4021 pad 1: +3V3D -> +3V3
- C4023 pad 1: +3V3D -> +3V3
- C4024 pad 1: +3V3D -> +3V3
- C4025 pad 1: +3V3D -> +3V3
- C5018 pad 1: /Control/Analog/ADC_N -> /Control/ADC/ADC_N
- C5018 pad 2: /Control/Analog/ADC_P -> /Control/ADC/ADC_P
- C6001 pad 2: /Control/ADC/CLK_DVDD -> +3V3
- C6002 pad 2: /Control/ADC/CLK_DVDD -> +3V3
- C6011 pad 2: +3V3D -> +3V3
- C6013 pad 2: +3V3D -> +3V3
- C7005 pad 1: +3V3D -> +3V3
- C7006 pad 1: +3V3D -> +3V3
- C8001 pad 1: +3V3D -> +3V3
- C8008 pad 1: /Power Input/VIN -> VIN
- C9001 pad 1: VIN_REF -> VIN
- C9002 pad 1: +12V -> /Power Rails/12_INT
- C9003 pad 1: +12V -> /Power Rails/12_INT
- C9004 pad 1: +12V -> /Power Rails/12_INT
- C9005 pad 1: +12V -> /Power Rails/12_INT
- C9006 pad 1: +12V -> /Power Rails/12_INT
- C9009 pad 1: +5V -> /Power Rails/5_INT
- C9010 pad 1: +1V0 -> /Power Rails/1_INT
- C9011 pad 2: +5V -> /Power Rails/5_INT
- C9012 pad 2: +5V -> /Power Rails/5_INT
- D8001 pad 1: /Power Input/VIN -> VIN
- FB3001 pad 2: +1V8D -> +1V8
- FB7001 pad 1: +3V3D -> +3V3
- FB7002 pad 1: +3V3D -> +3V3
- J3001 pad 1: +3V3D -> +3V3
- J3002 pad 1: +3V3D -> +3V3
- Q8001 pad 2: /Power Input/VIN -> VIN
- R3001 pad 1: +3V3D -> +3V3
- R3002 pad 1: +3V3D -> +3V3
- R3003 pad 1: +3V3D -> +3V3
- R3004 pad 1: +3V3D -> +3V3
- R3005 pad 1: +3V3D -> +3V3
- R3006 pad 1: +3V3D -> +3V3
- R3007 pad 1: +3V3D -> +3V3
- R3009 pad 1: +3V3D -> +3V3
- R3011 pad 1: +3V3D -> +3V3
- R3015 pad 2: +3V3D -> +3V3
- R5021 pad 1: /Control/Analog/ADC_P -> /Control/ADC/ADC_P
- R5022 pad 1: /Control/Analog/ADC_N -> /Control/ADC/ADC_N
- R8007 pad 1: /Power Input/VIN -> VIN
- R8014 pad 2: /Power Input/VIN -> VIN
- R9001 pad 2: +5V -> /Power Rails/5_INT
- R9003 pad 2: +1V0 -> /Power Rails/1_INT
- U3001 pad F10: +1V8D -> +1V8
- U3001 pad G13: +3V3D -> +3V3
- U3001 pad G2: +3V3D -> +3V3
- U3001 pad H10: +1V8D -> +1V8
- U3001 pad K10: +1V8D -> +1V8
- U3001 pad K13: +3V3D -> +3V3
- U3001 pad K2: +3V3D -> +3V3
- U3001 pad L9: +1V8D -> +1V8
- U3001 pad N13: +3V3D -> +3V3
- U3001 pad N2: +3V3D -> +3V3
- U3001 pad N6: +3V3D -> +3V3
- U3001 pad N7: +3V3D -> +3V3
- U3001 pad N8: +3V3D -> +3V3
- U3002 pad 8: +3V3D -> +3V3
- U3003 pad 1: +3V3D -> +3V3
- U3003 pad 16: +3V3D -> +3V3
- U3003 pad 7: +3V3D -> +3V3
- U5001 pad 1: /Control/Analog/ADC1_B -> /Control/Analog/ADC1_A
- U5001 pad 3: /Control/Analog/ADC1_A -> /Control/Analog/ADC1_B
- U6001 pad 1: /Control/ADC/CLK_DVDD -> +3V3
- U6001 pad 6: /Control/ADC/CLK_DVDD -> +3V3
- U6002 pad 13: +3V3D -> +3V3
- U8001 pad 1: +3V3D -> +3V3
- U8001 pad 2: GND -> SUPPLY_EN2
- U8001 pad 4: Net-(U8001-Pad4) -> GND
- U8001 pad 6: +5V -> Net-(U8001-Pad6)
- U8002 pad 5: Net-(U8001-Pad4) -> Net-(U8001-Pad7)
- U8002 pad 6: GND -> Net-(U8001-Pad6)
- U9001 pad 14: +12V -> /Power Rails/12_INT
- U9001 pad 22: VIN_REF -> VIN
- U9001 pad 23: VIN_REF -> VIN
- U9002 pad 1: VIN_REF -> VIN
- U9002 pad 5: +12V -> /Power Rails/12_INT
- U9003 pad 1: +12V -> /Power Rails/12_INT
- U9003 pad 2: +12V -> /Power Rails/12_INT
- U9003 pad 4: +5V -> /Power Rails/5_INT
- U9003 pad 5: +5V -> /Power Rails/5_INT
- U9004 pad 1: +12V -> /Power Rails/12_INT
- U9004 pad 2: +12V -> /Power Rails/12_INT
- U9004 pad 4: +1V0 -> /Power Rails/1_INT
- U9004 pad 5: +1V0 -> /Power Rails/1_INT
- U9005 pad 5: +5V -> /Power Rails/5_INT
- U9005 pad 8: +5V -> /Power Rails/5_INT
- U9006 pad 5: +5V -> /Power Rails/5_INT
- U9006 pad 8: +5V -> /Power Rails/5_INT
Routing:
- net GND: track 24.6 -> 41.1 mm, vias 8 -> 65
- net /Power Rails/5_INT: track 0.00 -> 10.1 mm, vias 0 -> 4
- net +1V8: track 0.00 -> 7.96 mm, vias 0 -> 8
- net +1V0: track 0.00 -> 7.78 mm, vias 0 -> 14
- net /Control/ADC/VREF: track 0.00 -> 4.84 mm, vias 0 -> 1
- net /Control/ADC/RBIAS: track 0.00 -> 3.73 mm
- net Net-(R9001-Pad1): track 0.00 -> 3.56 mm
- net Net-(R9003-Pad1): track 0.00 -> 3.56 mm
- net Net-(C9008-Pad1): track 0.00 -> 2.33 mm
- net Net-(C6003-Pad2): track 0.00 -> 2.31 mm
- net Net-(C9007-Pad1): track 0.00 -> 2.28 mm
- net /Control/ADC/VCM: track 0.00 -> 2.23 mm
- net Net-(C6004-Pad2): track 0.00 -> 1.93 mm
- net Net-(C9014-Pad2): track 0.00 -> 1.84 mm
- net Net-(C9013-Pad2): track 0.00 -> 1.84 mm
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- added copper zone on F.Cu, net +1V0
- added copper zone on In2.Cu, net +1V0
- added copper zone on F.Cu, net +1V8
- added copper zone on In2.Cu, net +1V8
- added copper zone on F.Cu, net +3V3
- added copper zone on F.Cu, net +5V
- added copper zone on F.Cu, net /Power Rails/12_INT
- added copper zone on F.Cu, net /Power Rails/5_INT
- added copper zone on F.Cu, net GND
- added copper zone on F.Cu, net Net-(C9015-Pad2)
- added copper zone on F.Cu, net Net-(C9016-Pad2)

Commit message: revised power input schematic
Parts:
- removed C8005, C8006, C8007: 0.47u, Capacitor_SMD:C_0402_1005Metric
- removed C8009: 10u, Capacitor_SMD:C_0603_1608Metric
- removed C8010: 0.47u, Capacitor_SMD:C_0603_1608Metric
- removed C8011: 1u, Capacitor_SMD:C_2220_5650Metric_Pad1.97x5.40mm_HandSolder
- removed FB8002: Ferrite_Bead_Small, Inductor_SMD:L_0805_2012Metric
- removed L8001: CM_CHOKE, wbraun_smd:744824622
- added FB11002: Ferrite_Bead_Small, Inductor_SMD:L_0805_2012Metric, F.Cu at (303.4, 67.8)
- added FB11003: Ferrite_Bead_Small, Inductor_SMD:L_0805_2012Metric, F.Cu at (303.4, 70.7)
- added FB12002: Ferrite_Bead_Small, Inductor_SMD:L_0805_2012Metric, F.Cu at (333.1, 47.2)
- added FB12003: Ferrite_Bead_Small, Inductor_SMD:L_0805_2012Metric, F.Cu at (333.1, 50.2)
- added FB13002: Ferrite_Bead_Small, Inductor_SMD:L_0805_2012Metric, F.Cu at (312.5, 67.8)
- added FB13003: Ferrite_Bead_Small, Inductor_SMD:L_0805_2012Metric, F.Cu at (316.9, 70.7)
- added FB14002: Ferrite_Bead_Small, Inductor_SMD:L_0805_2012Metric, F.Cu at (337.5, 59.1)
- added FB14003: Ferrite_Bead_Small, Inductor_SMD:L_0805_2012Metric, F.Cu at (333.1, 56.2)
- added J8002: mounting-hole-grounded, wbraun_smd:OMNI-UNI-30-50-D, F.Cu at (337.0, 79.5)
- added Q8003: Q_NMOS_GDS, Package_TO_SOT_THT:TO-247-3_Vertical, F.Cu at (299.6, 48.2)
- added R11005: 1, Resistor_SMD:R_0805_2012Metric, F.Cu at (299.0, 67.8)
- added R11006: 1, Resistor_SMD:R_0805_2012Metric, F.Cu at (299.0, 70.7)
- added R12005: 1, Resistor_SMD:R_0805_2012Metric, F.Cu at (337.5, 47.2)
- added R12006: 1, Resistor_SMD:R_0805_2012Metric, F.Cu at (337.5, 50.2)
- added R13005: 1, Resistor_SMD:R_0805_2012Metric, F.Cu at (312.5, 70.7)
- added R13006: 1, Resistor_SMD:R_0805_2012Metric, F.Cu at (316.9, 67.8)
- added R14005: 1, Resistor_SMD:R_0805_2012Metric, F.Cu at (333.1, 59.1)
- added R14006: 1, Resistor_SMD:R_0805_2012Metric, F.Cu at (337.5, 56.2)
- added REF**: TO-247-3_Horizontal_TabDown, Package_TO_SOT_THT:TO-247-3_Horizontal_TabDown, F.Cu at (213.8, 137.0)
- added REF**: TO-247-3_Horizontal_TabDown, Package_TO_SOT_THT:TO-247-3_Horizontal_TabDown, F.Cu at (190.0, 65.2)
- added REF**: TO-247-3_Horizontal_TabDown, Package_TO_SOT_THT:TO-247-3_Horizontal_TabDown, F.Cu at (213.8, 116.8)
- added REF**: 7693-term, wbraun_smd:7693-term, F.Cu at (177.5, 117.2)
- added REF**: 7693-term, wbraun_smd:7693-term, F.Cu at (177.8, 81.5)
- added REF**: TO-247-3_Horizontal_TabDown, Package_TO_SOT_THT:TO-247-3_Horizontal_TabDown, F.Cu at (190.0, 83.8)
- C8001: value 0.47u -> 4.7u; footprint Capacitor_SMD:C_0402_1005Metric -> Capacitor_SMD:C_0805_2012Metric
- C8004: value 10u -> 0.47u
- C8008: footprint Capacitor_THT:C_Rect_L31.5mm_W20.0mm_P27.50mm_MKS4 -> Capacitor_THT:C_Rect_L33.0mm_W13.0mm_P27.50mm_MKS4
- D8001: value D_Bridge_+AA- -> D; footprint wbraun_smd:Diode-GBJ-Vertical -> Package_TO_SOT_THT:TO-247-2_Vertical
- Q8002: value Q_NMOS_GDS -> 2N7002; footprint Package_TO_SOT_THT:TO-247-3_Vertical -> Package_TO_SOT_SMD:SOT-23
- R8001: value 10k -> 100; footprint Resistor_SMD:R_0603_1608Metric -> Resistor_SMD:R_0402_1005Metric
- R8002: value 4.7 -> 4.7K; footprint Resistor_SMD:R_0603_1608Metric -> Resistor_SMD:R_0402_1005Metric
- R8003: value 4.7 -> 100; footprint Resistor_SMD:R_0603_1608Metric -> Resistor_SMD:R_0402_1005Metric
- R8004: value 10k -> 4.7K; footprint Resistor_SMD:R_0603_1608Metric -> Resistor_SMD:R_0402_1005Metric
- R8005: value 10k -> 1; footprint Resistor_SMD:R_0603_1608Metric -> Resistor_SMD:R_0805_2012Metric
- R8006: value 4.7 -> 1; footprint Package_TO_SOT_THT:TO-247-2_Vertical -> Resistor_SMD:R_0805_2012Metric
- R8013: value 10k -> 4.7K
- U8001: value 74LVC2T45DC -> VOM1271; footprint Package_SO:VSSOP-8_2.3x2mm_P0.5mm -> Package_SO:SO-4_4.4x4.3mm_P2.54mm
- U8002: value ADuM5230 -> UCC5350SB; footprint Package_SO:SOIC-16W_7.5x10.3mm_P1.27mm -> Package_SO:SOIC-8_3.9x4.9mm_P1.27mm; moved to F.Cu
- moved C8001 321.6 mm to (307.8, 60.4)
- moved FB8001 303.7 mm to (316.4, 59.5)
- moved R8013 299.7 mm to (312.0, 60.2)
- moved R8003 271.2 mm to (324.1, 55.1)
- moved R8001 267.5 mm to (318.4, 62.0)
- moved R8002 266.1 mm to (315.4, 62.0)
- moved U8001 222.2 mm to (303.8, 23.8)
- moved Q8002 145.5 mm to (325.2, 48.0)
- moved C10007 132.4 mm to (335.5, 133.0)
- moved Q8001 131.5 mm to (352.5, 99.8)
- moved R8006 103.4 mm to (299.0, 60.4), turned to 0 degrees
- moved C10006 89.2 mm to (303.0, 88.8), turned to 270 degrees
- moved D8001 88.4 mm to (276.0, 48.8), turned to 0 degrees
- moved U8003 70.8 mm to (237.8, 179.5)
- moved U8002 66.2 mm to (318.4, 54.8)
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Connections:
- C10001 pad 1: /Inverter/VBUS -> VBUS
- C10001 pad 2: GNDPWR -> DRIVE_AUX-
- C10002 pad 1: /Inverter/VBUS -> VBUS
- C10002 pad 2: GNDPWR -> DRIVE_AUX-
- C10003 pad 1: /Inverter/VBUS -> VBUS
- C10003 pad 2: GNDPWR -> DRIVE_AUX-
- C10004 pad 1: /Inverter/VBUS -> VBUS
- C10004 pad 2: GNDPWR -> DRIVE_AUX-
- C10005 pad 1: /Inverter/VBUS -> VBUS
- C10005 pad 2: GNDPWR -> DRIVE_AUX-
- C10006 pad 1: /Inverter/VBUS -> VBUS
- C10007 pad 2: GNDPWR -> DRIVE_AUX-
- C8001 pad 1: +3V3 -> DRIVE_AUX+
- C8001 pad 2: GND -> DRIVE_AUX-
- C8002 pad 1: Net-(C8002-Pad1) -> VIN
- C8003 pad 2: Net-(C8003-Pad2) -> DRIVE_AUX-
- C8004 pad 1: +5V -> DRIVE_AUX+
- C8004 pad 2: GND -> DRIVE_AUX-
- C8008 pad 1: VIN -> /Power Input/S1
- C8008 pad 2: GNDPWR -> DRIVE_AUX-
- C9001 pad 2: GNDPWR -> DRIVE_AUX-
- C9017 pad 2: GNDPWR -> DRIVE_AUX-
- D8001 pad 1: VIN -> VBUS
- D8001 pad 2: Net-(C8002-Pad1) -> Net-(D8001-Pad2)
- F8001 pad 1: Net-(F8001-Pad1) -> VIN
- FB8001 pad 1: Net-(FB8001-Pad1) -> /Power Input/G2
- FB8001 pad 2: /Power Input/GATE1+ -> Net-(FB8001-Pad2)
- J8001 pad 1: Net-(J8001-Pad1) -> DRIVE_AUX-
- L8002 pad 2: SW_NODE -> Net-(D8001-Pad2)
- Q10001 pad DC+: /Inverter/VBUS -> VBUS
- Q10001 pad DC-: GNDPWR -> DRIVE_AUX-
- Q8001 pad 1: Net-(Q8001-Pad1) -> /Power Input/G1
- Q8001 pad 3: /Power Input/GATE- -> /Power Input/S1
- Q8002 pad 2: Net-(C8011-Pad2) -> GND
- Q8002 pad 3: /Power Input/GATE- -> Net-(Q8002-Pad3)
- R10001 pad 1: /Inverter/VBUS -> VBUS
- R10007 pad 2: GNDPWR -> DRIVE_AUX-
- R8001 pad 1: GND -> Net-(Q8002-Pad1)
- R8001 pad 2: SUPPLY_EN1 -> Net-(R8001-Pad2)
- R8002 pad 1: Net-(Q8001-Pad1) -> Net-(Q8002-Pad1)
- R8002 pad 2: Net-(FB8001-Pad1) -> GND
- R8003 pad 1: Net-(Q8002-Pad1) -> Net-(R8003-Pad1)
- R8003 pad 2: Net-(FB8002-Pad1) -> +3V3
- R8004 pad 1: Net-(Q8001-Pad1) -> GND
- R8004 pad 2: /Power Input/GATE- -> SUPPLY_EN1
- R8005 pad 1: Net-(Q8002-Pad1) -> Net-(FB8001-Pad2)
- R8005 pad 2: /Power Input/GATE- -> Net-(R8005-Pad2)
- R8006 pad 1: /Power Input/GATE- -> Net-(FB8001-Pad2)
- R8006 pad 2: Net-(C8011-Pad1) -> Net-(R8006-Pad2)
- R8011 pad 2: GNDPWR -> DRIVE_AUX-
- R8013 pad 1: SUPPLY_EN2 -> DRIVE_AUX-
- R8013 pad 2: GND -> /Power Input/G2
- R8014 pad 1: /Power Input/GATE- -> /Power Input/S1
- R9010 pad 2: GNDPWR -> DRIVE_AUX-
- U8001 pad 1: +3V3 -> Net-(R8003-Pad1)
- U8001 pad 2: SUPPLY_EN2 -> Net-(Q8002-Pad3)
- U8001 pad 3: SUPPLY_EN1 -> /Power Input/S1
- U8001 pad 4: GND -> /Power Input/G1
- U8002 pad 1: GND -> +3V3
- U8002 pad 2: +5V -> SUPPLY_EN1
- U8002 pad 3: Net-(U8002-Pad3) -> GND
- U8002 pad 5: Net-(U8001-Pad7) -> DRIVE_AUX+
- U8002 pad 6: Net-(U8001-Pad6) -> Net-(R8005-Pad2)
- U8002 pad 7: +5V -> Net-(R8006-Pad2)
- U8002 pad 8: GND -> DRIVE_AUX-
- U8003 pad 1: Net-(C8011-Pad2) -> /Power Input/S1
- U8003 pad 2: Net-(C8011-Pad2) -> /Power Input/S1
- U9001 pad 1: GNDPWR -> DRIVE_AUX-
- U9001 pad 2: GNDPWR -> DRIVE_AUX-
- U9001 pad 3: GNDPWR -> DRIVE_AUX-
- U9002 pad 2: GNDPWR -> DRIVE_AUX-
Routing:
- added copper zone on F.Cu, net VBUS
- removed copper zone on In2.Cu, net /Inverter/Out2
- removed copper zone on F.Cu, net /Inverter/VBUS
- removed copper zone on B.Cu, net SW_NODE

Commit message: routing, all componens placed on PCB
Parts:
- removed C10006: 33n, Capacitor_THT:C_Rect_L18.0mm_W7.0mm_P15.00mm_FKS3_FKP3
- removed C3002, C4020, C4021: 0.47u, Capacitor_SMD:C_0402_1005Metric
- removed C5008, C5012: 4.7u, Capacitor_SMD:C_0402_1005Metric
- removed C9002, C9003: 10u, Capacitor_SMD:C_1206_3216Metric
- removed FB11002, FB11003, FB13002, FB13003, FB14002, FB14003: Ferrite_Bead_Small, Inductor_SMD:L_0805_2012Metric
- removed J8002: mounting-hole-grounded, wbraun_smd:OMNI-UNI-30-50-D
- removed L5001: CM_CHOKE, wbraun_smd:SRF2012
- removed R10005, R10006, R8008, R8009: R, Resistor_SMD:R_0805_2012Metric
- removed R10008, R8012: R, Resistor_SMD:R_0603_1608Metric
- removed R11005, R11006, R13005, R13006, R14005, R14006: 1, Resistor_SMD:R_0805_2012Metric
- removed REF** (x4): TO-247-3_Horizontal_TabDown, Package_TO_SOT_THT:TO-247-3_Horizontal_TabDown
- removed REF** (x2): 7693-term, wbraun_smd:7693-term
- added C4026: 0.47u, Capacitor_SMD:C_0402_1005Metric, B.Cu at (92.5, 117.2)
- added C8005: 0.47u, Capacitor_SMD:C_0603_1608Metric, B.Cu at (228.8, 114.0)
- added J10002: Conn_01x01_Female, wbraun_smd:7693-term, F.Cu at (177.0, 80.5)
- added R5020: 33, Resistor_SMD:R_0402_1005Metric, F.Cu at (97.0, 144.0)
- added R5023: 33, Resistor_SMD:R_0402_1005Metric, F.Cu at (97.0, 145.2)
- C3001, C4005, C4007, C4008, C4009, C4010, C4011, C4012, C4013, C4014, C4015, C4016, C4017, C4018, C4019, C4022, C4024, C4025, FB12002, FB12003, R10001, R10002, R10003, R10004, R12005, R12006, R8007, R8010, R8011: moved to B.Cu
- C8003: value 33n -> 0.47u; footprint Capacitor_THT:C_Rect_L18.0mm_W7.0mm_P15.00mm_FKS3_FKP3 -> Capacitor_SMD:C_0603_1608Metric
- D3001, D3002: footprint wbraun_smd:LED-T1-RIGHT-ANGLE_4.6x4.4mm -> LED_SMD:LED_0805_2012Metric
- D8001, R8014: footprint Package_TO_SOT_THT:TO-247-2_Vertical -> wbraun_smd:TO-247_2_horizontal_under
- FB3001, FB3002: value FB -> Ferrite_Bead_Small; footprint Inductor_SMD:L_0805_2012Metric -> Inductor_SMD:L_0402_1005Metric; moved to B.Cu
- J10001: value Conn_01x02_Female -> Conn_01x01_Female; footprint wbraun_smd:Anderson_PP45_2x1 -> wbraun_smd:7693-term
- Q8001, Q8003: footprint Package_TO_SOT_THT:TO-247-3_Vertical -> wbraun_smd:TO-247_3_horizontal_under
- R10007: footprint Resistor_SMD:R_0603_1608Metric -> Resistor_SMD:R_0805_2012Metric; moved to B.Cu
- moved R10007 278.6 mm to (230.8, 101.8)
- moved R10004 277.1 mm to (227.2, 101.8)
- moved R10003 272.2 mm to (223.8, 101.8)
- moved R10001 269.2 mm to (216.8, 101.8)
- moved R10002 235.7 mm to (220.2, 101.8)
- moved Q8002 230.8 mm to (104.0, 114.0), turned to 270 degrees
- moved R8011 226.2 mm to (230.8, 97.5)
- moved R12006 226.2 mm to (127.0, 133.0), turned to 90 degrees
- moved R12005 225.2 mm to (129.2, 133.0), turned to 270 degrees
- moved R8007 223.1 mm to (223.8, 97.5)
- moved FB12003 220.8 mm to (127.0, 129.2), turned to 90 degrees
- moved R8001 220.2 mm to (103.5, 110.2), turned to 180 degrees
- moved FB12002 219.7 mm to (129.2, 129.2), turned to 90 degrees
- moved R8002 217.6 mm to (103.5, 111.5), turned to 180 degrees
- moved U5003 174.4 mm to (96.2, 141.2)
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Connections:
- C10001 pad 2: DRIVE_AUX- -> PWRGND
- C10002 pad 2: DRIVE_AUX- -> PWRGND
- C10003 pad 2: DRIVE_AUX- -> PWRGND
- C10004 pad 2: DRIVE_AUX- -> PWRGND
- C10005 pad 2: DRIVE_AUX- -> PWRGND
- C10007 pad 2: DRIVE_AUX- -> PWRGND
- C3001 pad 1: /Control/FPGA/VDDA -> /Control/FPGA/VCCADC
- C3001 pad 2: /Control/FPGA/GNDA -> /Control/FPGA/GNDADC
- C5010 pad 1: VIN_SENSE -> Net-(C5010-Pad1)
- C5011 pad 2: VBUS_SENSE -> Net-(C5011-Pad2)
- C5015 pad 1: Net-(C5015-Pad1) -> TEMP_B
- C8001 pad 2: DRIVE_AUX- -> PWRGND
- C8002 pad 2: Earth -> PWRGND
- C8003 pad 1: Earth -> +3V3
- C8003 pad 2: DRIVE_AUX- -> GND
- C8004 pad 2: DRIVE_AUX- -> PWRGND
- C8008 pad 2: DRIVE_AUX- -> PWRGND
- C9001 pad 2: DRIVE_AUX- -> PWRGND
- C9017 pad 2: DRIVE_AUX- -> PWRGND
- FB3001 pad 1: /Control/FPGA/VDDA -> /Control/FPGA/GNDADC
- FB3001 pad 2: +1V8 -> GND
- FB3002 pad 1: GND -> /Control/FPGA/VCCADC
- FB3002 pad 2: /Control/FPGA/GNDA -> +1V8
- J10001 pad 1: /Inverter/Out2 -> /Inverter/Out1
- J8001 pad 1: DRIVE_AUX- -> PWRGND
- Q10001 pad AC1: SW_NODE -> /Inverter/Out1
- Q10001 pad DC-: DRIVE_AUX- -> PWRGND
- Q10001 pad T1: TEMP_A -> GND
- Q8003 pad 3: DRIVE_AUX- -> PWRGND
- R10004 pad 2: Net-(R10004-Pad2) -> VBUS_SENSE
- R10007 pad 1: Net-(R10006-Pad2) -> VBUS_SENSE
- R10007 pad 2: DRIVE_AUX- -> PWRGND
- R12006 pad 1: DRIVE_AUX- -> PWRGND
- R5019 pad 1: Net-(C5015-Pad1) -> TEMP_B
- R8010 pad 1: Net-(R8009-Pad2) -> Net-(R8007-Pad2)
- R8010 pad 2: Net-(R8010-Pad2) -> VIN_SENSE
- R8011 pad 1: Net-(R8010-Pad2) -> VIN_SENSE
- R8011 pad 2: DRIVE_AUX- -> PWRGND
- R8013 pad 1: DRIVE_AUX- -> PWRGND
- R9010 pad 2: DRIVE_AUX- -> PWRGND
- U3001 pad B1: FIBER_TX -> Net-(U3001-PadB1)
- U3001 pad B14: GATE_1 -> ADC_CSB
- U3001 pad C1: FIBER_RX -> Net-(U3001-PadC1)
- U3001 pad C14: Net-(U3001-PadC14) -> ADC_SCLK
- U3001 pad D12: Net-(U3001-PadD12) -> ADC_SDIO
- U3001 pad D13: Net-(U3001-PadD13) -> ADC_D0
- U3001 pad D14: GATE_2 -> ADC_D1
- U3001 pad E12: Net-(U3001-PadE12) -> ADC_D2
- U3001 pad E13: Net-(U3001-PadE13) -> ADC_D3
- U3001 pad F12: Net-(U3001-PadF12) -> ADC_D4
- U3001 pad F13: Net-(U3001-PadF13) -> ADC_D5
- U3001 pad F14: GATE_3 -> ADC_D6
- U3001 pad F7: /Control/FPGA/GNDA -> /Control/FPGA/GNDADC
- U3001 pad F8: /Control/FPGA/VDDA -> /Control/FPGA/VCCADC
- U3001 pad G14: /Control/FPGA/DEBUG_TX -> ADC_D7
- U3001 pad G7: /Control/FPGA/GNDA -> GND
- U3001 pad H12: /Control/FPGA/DEBUG_RX -> Net-(U3001-PadH12)
- U3001 pad H13: UVLO -> ADC_D9
- U3001 pad H14: GATE_4 -> ADC_D8
- U3001 pad H8: /Control/FPGA/GNDA -> GND
- U3001 pad J12: /Control/FPGA/LED2 -> Net-(U3001-PadJ12)
- U3001 pad J13: /Control/FPGA/LED1 -> Net-(U3001-PadJ13)
- U3001 pad J14: ADC_D0 -> ADC_MODE
- U3001 pad K12: ZCS_DETECT -> Net-(U3001-PadK12)
- U3001 pad L13: ADC_D2 -> Net-(U3001-PadL13)
- U3001 pad L14: ADC_D1 -> Net-(U3001-PadL14)
- U3001 pad M13: ADC_D4 -> Net-(U3001-PadM13)
- U3001 pad M14: ADC_D3 -> Net-(U3001-PadM14)
- U3001 pad M2: ADC_MODE -> Net-(U3001-PadM2)
- U3001 pad N1: ADC_SDIO -> Net-(U3001-PadN1)
- U3001 pad N11: ADC_D8 -> Net-(U3001-PadN11)
- U3001 pad N14: ADC_D5 -> Net-(U3001-PadN14)
- U3001 pad P11: ADC_D9 -> Net-(U3001-PadP11)
- U3001 pad P12: ADC_D7 -> Net-(U3001-PadP12)
- U3001 pad P13: ADC_D6 -> Net-(U3001-PadP13)
- U3001 pad P2: ADC_SCLK -> Net-(U3001-PadP2)
- U3001 pad P3: ADC_CSB -> Net-(U3001-PadP3)
- U5003 pad 1: VIN_SENSE -> Net-(C5010-Pad1)
- U5003 pad 3: VBUS_SENSE -> Net-(C5011-Pad2)
- U5004 pad 3: Net-(C5015-Pad1) -> TEMP_B
- U8002 pad 8: DRIVE_AUX- -> PWRGND
- U9001 pad 1: DRIVE_AUX- -> PWRGND
- U9001 pad 2: DRIVE_AUX- -> PWRGND
- U9001 pad 3: DRIVE_AUX- -> PWRGND
- U9002 pad 2: DRIVE_AUX- -> PWRGND
Routing:
- net GND: track 41.1 -> 96.5 mm, vias 65 -> 111
- net +3V3: track 15.3 -> 40.1 mm, vias 7 -> 27
- net /Control/FPGA/TCK: track 0.00 -> 22.3 mm
- net /Control/FPGA/FLASH_SCK: track 0.00 -> 20.4 mm
- net /Control/FPGA/FLASH_IO0: track 0.00 -> 18.4 mm, vias 0 -> 2
- net /Control/FPGA/FLASH_IO2: track 0.00 -> 18.3 mm
- net /Control/FPGA/FLASH_IO3: track 0.00 -> 16.6 mm
- net ADC_DCO: track 0.00 -> 14.7 mm
- net ADC_D9: track 0.00 -> 12.1 mm
- net ADC_D5: track 0.00 -> 11.4 mm
- net +1V8: track 7.96 -> 18.9 mm, vias 8 -> 12
- net ADC_D2: track 0.00 -> 10.9 mm
- net ADC_D6: track 0.00 -> 10.9 mm
- net ADC_D7: track 0.00 -> 10.8 mm
- net ADC_D4: track 0.00 -> 10.6 mm
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- added copper zone on In1.Cu, net GND
Other:
- net class Default: clearance 0.153 -> 0.1; trace_width 0.153 -> 0.1; via_dia 0.6 -> 0.5; via_drill 0.3 -> 0.2
- rule trace_clearance: 0.153 -> 0.1
- rule trace_min: 0.153 -> 0.1
- rule via_min_drill: 0.3 -> 0.2
- rule via_min_size: 0.4 -> 0.5

Commit message: routing progress
Parts:
- removed C5016: 4.7u, Capacitor_SMD:C_0402_1005Metric
- C5009: moved to F.Cu
- C5014: value 4.7u -> 0.47u
- FB7001, FB7002: footprint Inductor_SMD:L_0805_2012Metric -> Inductor_SMD:L_0402_1005Metric
- J8001: value Conn_01x02_Female -> Conn_01x03_Female; footprint wbraun_smd:Anderson_PP45_2x1 -> wbraun_smd:Terminal-block-plug_3x1_5mm-pitch
- moved R10001 50.0 mm to (258.5, 129.2)
- moved R10002 50.0 mm to (262.0, 129.2)
- moved R10003 50.0 mm to (265.5, 129.2)
- moved R10004 50.0 mm to (269.0, 129.2)
- moved R10007 50.0 mm to (272.5, 129.2)
- moved R8007 50.0 mm to (265.5, 125.0)
- moved R8010 50.0 mm to (269.0, 125.0)
- moved R8011 50.0 mm to (272.5, 125.0)
- moved F8001 26.3 mm to (231.0, 79.5), turned to 90 degrees
- moved U8001 23.8 mm to (198.2, 97.8), turned to 90 degrees
- moved R5019 23.7 mm to (100.5, 130.0)
- moved R5016 22.5 mm to (107.2, 130.0)
- moved C5017 22.3 mm to (106.0, 130.0), turned to 270 degrees
- moved U5004 21.6 mm to (103.2, 131.2)
- moved C5015 21.4 mm to (100.5, 132.0)
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Connections:
- J8001 pad 1: PWRGND -> Net-(F8001-Pad2)
- J8001 pad 2: Net-(F8001-Pad2) -> PWRGND
Routing:
- net /Inverter/Gate Drive 2/Source: track 10.1 -> 62.8 mm
- net /Inverter/Gate Drive 4/Source: track 10.1 -> 60.5 mm, vias 2 -> 3
- net /Inverter/Gate Drive 2/Gate: track 0.00 -> 45.9 mm
- net /Inverter/Gate Drive 4/Gate: track 0.00 -> 42.8 mm
- net Net-(J5001-Pad1): track 0.00 -> 20.5 mm
- net /Inverter/Gate Drive 1/Gate: track 0.00 -> 17.9 mm
- net GND: track 96.5 -> 114.4 mm, vias 111 -> 130
- net /Inverter/Gate Drive 3/Gate: track 0.00 -> 15.8 mm
- net /Inverter/Gate Drive 1/Source: track 10.1 -> 23.5 mm
- net /Inverter/Gate Drive 3/Source: track 10.1 -> 23.5 mm
- net /Control/Analog/ADC1_MUXED: track 0.00 -> 11.7 mm
- net +3V3: track 40.1 -> 51.2 mm, vias 27 -> 36
- net /Inverter/Gate Drive 1/V+: track 4.78 -> 15.5 mm
- net /Inverter/Gate Drive 3/V+: track 4.78 -> 14.8 mm
- net /Inverter/Gate Drive 4/V+: track 4.78 -> 14.6 mm
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- added copper zone on B.Cu, net /Inverter/Out1
- added copper zone on B.Cu, net /Inverter/Out2
- added copper zone on B.Cu, net /Power Input/S1
- added copper zone on B.Cu, net VIN
Other:
- rule pad_to_mask_clearance: 0.051 -> 0.05
