File: pcb/integrated/Interface.sch (KiCad schematic (older format))
At the start: 10 parts, among them U7001 AFBR-1624Z, U7002 AFBR-2624Z

Commit message: schematic fixes and component placement
Connections:
- net +3V3D renamed +3V3
Changed lines of the file:
@@
 Wire Wire Line
 	5500 4150 5500 4350
-Text GLabel 5500 2350 2    50   Input ~ 0
-+3V3D
-Text GLabel 5500 3650 2    50   Input ~ 0
-+3V3D
 Wire Wire Line
 	3700 3850 3800 3850
@@
 	3800 3850 3800 3950
 Connection ~ 3800 3950
+$Comp
+L power:+3V3 #PWR0175
+U 1 1 5D8191B5
+P 5500 2350
+F 0 "#PWR0175" H 5500 2200 50  0001 C CNN
+F 1 "+3V3" H 5515 2523 50  0000 C CNN
+F 2 "" H 5500 2350 50  0001 C CNN
+F 3 "" H 5500 2350 50  0001 C CNN
+	1    5500 2350
+	1    0    0    -1
+$EndComp
+$Comp
+L power:+3V3 #PWR0176
+U 1 1 5D819925
+P 5500 3650
+F 0 "#PWR0176" H 5500 3500 50  0001 C CNN
+F 1 "+3V3" H 5515 3823 50  0000 C CNN
+F 2 "" H 5500 3650 50  0001 C CNN
+F 3 "" H 5500 3650 50  0001 C CNN
+	1    5500 3650
+	1    0    0    -1
+$EndComp
 $EndSCHEMATC

Commit message: routing progress
Parts:
- FB7001, FB7002: footprint Inductor_SMD:L_0805_2012Metric -> Inductor_SMD:L_0402_1005Metric
Changed lines of the file:
@@
 F 0 "FB7001" V 4776 2450 50  0000 C CNN
 F 1 "Ferrite_Bead" V 4867 2450 50  0000 C CNN
-F 2 "Inductor_SMD:L_0805_2012Metric" V 4980 2450 50  0001 C CNN
+F 2 "Inductor_SMD:L_0402_1005Metric" V 4980 2450 50  0001 C CNN
 F 3 "~" H 5050 2450 50  0001 C CNN
 	1    5050 2450
@@
 $EndComp
 $Comp
-L Device:Ferrite_Bead FB7002
-U 1 1 5C606F0D
-P 5050 3750
-F 0 "FB7002" V 4776 3750 50  0000 C CNN
-F 1 "Ferrite_Bead" V 4867 3750 50  0000 C CNN
-F 2 "Inductor_SMD:L_0805_2012Metric" V 4980 3750 50  0001 C CNN
-F 3 "~" H 5050 3750 50  0001 C CNN
-	1    5050 3750
-	0    1    1    0
-$EndComp
-$Comp
 L Device:C C7004
 U 1 1 5C606F13
@@
 	1    0    0    -1
 $EndComp
+$Comp
+L Device:Ferrite_Bead FB7002
+U 1 1 5C606F0D
+P 5050 3750
+F 0 "FB7002" V 4776 3750 50  0000 C CNN
+F 1 "Ferrite_Bead" V 4867 3750 50  0000 C CNN
+F 2 "Inductor_SMD:L_0402_1005Metric" V 4980 3750 50  0001 C CNN
+F 3 "~" H 5050 3750 50  0001 C CNN
+	1    5050 3750
+	0    1    1    0
+$EndComp
 $EndSCHEMATC
