File: pcb/integrated/PoweInput.sch (KiCad schematic (older format))
At the start: 28 parts, among them J8001 Conn_01x03_Female, Q8001 Q_NMOS_GDS, Q8002 2N7002, Q8003 Q_NMOS_GDS, U8001 VOM1271, U8002 UCC5350SB, U8003 ACS730

Commit message: updated component values for schematic
Parts:
- C8002: value 33n -> B32922C3224M189
- C8008: value 22u -> C4AQLBU5100A1XK
- Q8001, Q8003: value Q_NMOS_GDS -> STW40N65M2
- Q8002: value 2N7002 -> FDV301N
- R8007, R8010: value R -> 470k
- R8011: value R -> 3.16k
- U8002: value UCC5350SB -> UCC5390SC
- U8003: value ACS730 -> ACS730KLCTR-20AB-T
- renumbered D8001 to IDWD10G120C5XKSA1
Changed lines of the file:
@@
 EESchema Schematic File Version 4
 LIBS:integrated-cache
-EELAYER 30 0
+EELAYER 26 0
 EELAYER END
 $Descr A4 11693 8268
@@
 AR Path="/5D688380/5D688D57" Ref="C8002"  Part="1"
 F 0 "C8002" H 2565 2346 50  0000 L CNN
-F 1 "33n" H 2565 2255 50  0000 L CNN
+F 1 "B32922C3224M189" H 2565 2255 50  0000 L CNN
 F 2 "Capacitor_THT:C_Rect_L18.0mm_W7.0mm_P15.00mm_FKS3_FKP3" H 2488 2150 50  0001 C CNN
 F 3 "~" H 2450 2300 50  0001 C CNN
@@
 AR Path="/5D688380/5D688D9E" Ref="C8008"  Part="1"
 F 0 "C8008" H 5215 2546 50  0000 L CNN
-F 1 "22u" H 5215 2455 50  0000 L CNN
+F 1 "C4AQLBU5100A1XK" H 5100 2800 50  0000 L CNN
 F 2 "Capacitor_THT:C_Rect_L33.0mm_W13.0mm_P27.50mm_MKS4" H 5138 2350 50  0001 C CNN
 F 3 "~" H 5100 2500 50  0001 C CNN
@@
 AR Path="/5D688380/5D8E4443" Ref="R8007"  Part="1"
 F 0 "R8007" H 9770 2796 50  0000 L CNN
-F 1 "R" H 9770 2705 50  0000 L CNN
+F 1 "470k" H 9770 2705 50  0000 L CNN
 F 2 "Resistor_SMD:R_0805_2012Metric" V 9630 2750 50  0001 C CNN
 F 3 "~" H 9700 2750 50  0001 C CNN
@@
 AR Path="/5D688380/5D8E4458" Ref="R8010"  Part="1"
 F 0 "R8010" H 9770 3196 50  0000 L CNN
-F 1 "R" H 9770 3105 50  0000 L CNN
+F 1 "470k" H 9770 3105 50  0000 L CNN
 F 2 "Resistor_SMD:R_0805_2012Metric" V 9630 3150 50  0001 C CNN
 F 3 "~" H 9700 3150 50  0001 C CNN
@@
 AR Path="/5D688380/5D8E446D" Ref="R8011"  Part="1"
 F 0 "R8011" H 9770 3796 50  0000 L CNN
-F 1 "R" H 9770 3705 50  0000 L CNN
+F 1 "3.16k" H 9770 3705 50  0000 L CNN
 F 2 "Resistor_SMD:R_0805_2012Metric" V 9630 3750 50  0001 C CNN
 F 3 "~" H 9700 3750 50  0001 C CNN
@@
 P 3550 2450
 F 0 "Q8001" H 3755 2496 50  0000 L CNN
-F 1 "Q_NMOS_GDS" H 3755 2405 50  0000 L CNN
+F 1 "STW40N65M2" H 3755 2405 50  0000 L CNN
 F 2 "wbraun_smd:TO-247_3_horizontal_under" H 3750 2550 50  0001 C CNN
 F 3 "~" H 3550 2450 50  0001 C CNN
@@
 VIN
 $Comp
-L Device:D D8001
+L Device:D IDWD10G120C5XKSA1
 U 1 1 5DB78EFD
 P 8050 2100
-F 0 "D8001" V 8004 2179 50  0000 L CNN
-F 1 "D" V 8095 2179 50  0000 L CNN
+F 0 "IDWD10G120C5XKSA1" H 7650 1900 50  0000 L CNN
+F 1 "D" H 8150 2200 50  0000 L CNN
 F 2 "wbraun_smd:TO-247_2_horizontal_under" H 8050 2100 50  0001 C CNN
 F 3 "~" H 8050 2100 50  0001 C CNN
@@
 P 7350 2650
 F 0 "Q8003" H 7555 2696 50  0000 L CNN
-F 1 "Q_NMOS_GDS" H 7555 2605 50  0000 L CNN
+F 1 "STW40N65M2" H 7555 2605 50  0000 L CNN
 F 2 "wbraun_smd:TO-247_3_horizontal_under" H 7550 2750 50  0001 C CNN
 F 3 "~" H 7350 2650 50  0001 C CNN
@@
 P 6250 2700
 F 0 "U8003" H 6250 3165 50  0000 C CNN
-F 1 "ACS730" H 6250 3074 50  0000 C CNN
+F 1 "ACS730KLCTR-20AB-T" H 6250 3074 50  0000 C CNN
 F 2 "Package_SO:SOIC-8_3.9x4.9mm_P1.27mm" H 5950 2800 50  0001 C CNN
 F 3 "" H 5950 2800 50  0001 C CNN
@@
 AR Path="/5D688380/5DC0C4B1" Ref="U8002"  Part="1"
 F 0 "U8002" H 4350 6465 50  0000 C CNN
-F 1 "UCC5350SB" H 4350 6374 50  0000 C CNN
+F 1 "UCC5390SC" H 4350 6374 50  0000 C CNN
 F 2 "Package_SO:SOIC-8_3.9x4.9mm_P1.27mm" H 4000 6100 50  0001 C CNN
 F 3 "" H 4000 6100 50  0001 C CNN
@@
 P 2450 4750
 F 0 "Q8002" H 2656 4796 50  0000 L CNN
-F 1 "2N7002" H 2656 4705 50  0000 L CNN
+F 1 "FDV301N" H 2656 4705 50  0000 L CNN
 F 2 "Package_TO_SOT_SMD:SOT-23" H 2650 4675 50  0001 L CIN
 F 3 "https://www.fairchildsemi.com/datasheets/2N/2N7002.pdf" H 2450 4750 50  0001 L CNN
